File: Enceinte/Enceinte.kicad_sch (KiCad schematic)
At the start: 17 parts, among them J1 Conn_01x07, J2 Conn_01x02, J3 Conn_01x02, J4 Conn_01x02, J5 Conn_01x02, J6 Conn_01x05, J7 Conn_01x06, J8 Conn_01x02, J9 Conn_01x02, U1 173010342

Commit message: Changement régulateur de tension
Parts:
- removed C1, C4: 4u7, Capacitor_SMD:C_0805_2012Metric, symbol Device:C
- removed C2, C3: 100 n, Capacitor_SMD:C_0402_1005Metric, symbol Device:C
- removed J6: Conn_01x05, Connector_PinSocket_2.54mm:PinSocket_1x05_P2.54mm_Vertical, symbol Connector_Generic:Conn_01x05
- removed U1: 173010342, MagIC_THT_Wurth:U_Wurth_MagIC-FDSM_173010x42, symbol MagIC_Wurth_MagIC-FDSM:173010342
- added C3: 0.1u, Capacitor_SMD:C_0603_1608Metric, symbol Device:C_Small
- added C4: 0.33u, Capacitor_SMD:C_0603_1608Metric, symbol Device:C_Small
- added H1, H2, H3, H4: MountingHole_Pad, MountingHole:MountingHole_2.5mm_Pad, symbol Mechanical:MountingHole_Pad
- added U1: L7805, L7805:TO255P1020X450X2000-3, symbol Regulator_Linear:L7805
Connections:
- net BT D is gone; now on net In_Pot_R: J1.4 (Pin_4)
- net BT G is gone; now on net In_Pot_L: J1.5 (Pin_5)
- net +12V: now also C4.1, U1.1 (IN)
- net +5V: now also C3.1, U1.3 (OUT)
- net GND: now also C3.2, C4.2, U1.2 (GND)
Other:
- note removed: "Alimentation 5V"
- note removed: "Jack à coupure"
- moved on the sheet: J1, J2, J3, J4, J5, J8, J9, R1, R2, R3

Commit message: des changements sont à faire
Parts:
- removed J1: Conn_01x07, Connector_PinSocket_2.54mm:PinSocket_1x07_P2.54mm_Vertical, symbol Connector_Generic:Conn_01x07
- removed U1: L7805, L7805:TO255P1020X450X2000-3, symbol Regulator_Linear:L7805
- added C1: 0.1u, Capacitor_SMD:C_0603_1608Metric, symbol Device:C_Small
- added J6: Conn_01x06, Connector_PinSocket_2.54mm:PinSocket_1x06_P2.54mm_Vertical, symbol Connector_Generic:Conn_01x06
- added L5: L_Small, symbol Device:L_Small
- added U2: AZ1117CH2-5.0, Package_TO_SOT_SMD:SOT-223-3_TabPin2, symbol Regulator_Linear:AZ1117CH2-5.0
Connections:
- net +12V: no longer C4.1
- net +5V: now also J6.3 (Pin_3), U2.3 (OUT)
- net GND: now also C1.2, J6.4 (Pin_4), U2.2 (GND)
- net In_Pot_L: now also J6.5 (Pin_5)
- net In_Pot_R: now also J6.6 (Pin_6)
- net at J2.2 (Pin_2), R1.1, R2.1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: now also J6.1 (Pin_1)
- new net: C1.1, L5.1
- new net: C4.1, L5.2, U2.1 (IN)
Other:
- moved on the sheet: C3, C4, J2, J3, J4, J5, R1, R2, R3

Commit message: doc latex
Parts:
- removed C1, C3: 0.1u, Capacitor_SMD:C_0603_1608Metric, symbol Device:C_Small
- removed C4: 0.33u, Capacitor_SMD:C_0603_1608Metric, symbol Device:C_Small
- removed L5: L_Small, symbol Device:L_Small
- removed U2: AZ1117CH2-5.0, Package_TO_SOT_SMD:SOT-223-3_TabPin2, symbol Regulator_Linear:AZ1117CH2-5.0
- added C1: 100n, Capacitor_SMD:C_0603_1608Metric, symbol Device:C
- added C2, C3, C6: 4u7, Capacitor_SMD:C_0603_1608Metric, symbol Device:C
- added C4, C5: 100 n, Capacitor_SMD:C_0603_1608Metric, symbol Device:C
- added D1: LED, LED_SMD:LED_0603_1608Metric, symbol Device:LED
- added L1: 100n, Inductor_SMD:L_0603_1608Metric, symbol Device:L_Small
- added R8: 1k, Resistor_SMD:R_0402_1005Metric, symbol Device:R
- added TP1: TestPoint, TestPoint:TestPoint_Pad_D1.5mm, symbol Connector:TestPoint
- added U1: 173010342, MagIC_THT_Wurth:U_Wurth_MagIC-FDSM_173010x42, symbol MagIC_Wurth_MagIC-FDSM:173010342
- J1: renamed from J6; footprint Connector_PinSocket_2.54mm:PinSocket_1x06_P2.54mm_Vertical -> Connector_JST:JST_XH_B6B-XH-A_1x06_P2.50mm_Vertical
- J2, J3, J4, J5: footprint Connector_PinSocket_2.54mm:PinSocket_1x02_P2.54mm_Vertical -> Connector_JST:JST_XH_B2B-XH-A_1x02_P2.50mm_Vertical
- J6: renamed from J8; footprint Connector_PinSocket_2.54mm:PinSocket_1x02_P2.54mm_Vertical -> Connector_JST:JST_XH_B2B-XH-A_1x02_P2.50mm_Vertical
- J7: renamed from J9; footprint Connector_PinSocket_2.54mm:PinSocket_1x02_P2.54mm_Vertical -> Connector_JST:JST_XH_B2B-XH-A_1x02_P2.50mm_Vertical
- J8: renamed from J7; footprint Connector_PinSocket_2.54mm:PinSocket_1x06_P2.54mm_Vertical -> Connector_JST:JST_XH_B6B-XH-A_1x06_P2.50mm_Vertical
Connections:
- net +12V: now also C1.2, C2.1, L1.1
- net +5V: now also C5.1, C6.1, R8.1, TP1.1, U1.3 (VOUT)
- net GND: now also H1.1, H2.1, H3.1, H4.1, C1.1, C2.2, C3.2, C4.2, C5.2, C6.2, D1.1 (K), U1.2 (GND)
- new net: C3.1, C4.1, L1.2, U1.1 (VIN)
- new net: D1.2 (A), R8.2
Other:
- note added: "Regulateur"
- note removed: "Power Switch"
- moved on the sheet: H1, H2, H3, H4

Commit message: nouvelles inductances
Parts:
- L1: footprint Inductor_SMD:L_0603_1608Metric -> Library_inductance_new:CWF1612A100J
Changed lines of the file:
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@@
 			)
 		)
-		(property "Footprint" "Inductor_SMD:L_0603_1608Metric"
+		(property "Footprint" "Library_inductance_new:CWF1612A100J"
 			(at 45.72 151.13 0)
 			(effects

Commit message: indu Wurth
Parts:
- removed TP1: TestPoint, TestPoint:TestPoint_Pad_D1.5mm, symbol Connector:TestPoint
- L1: footprint Library_inductance_new:CWF1612A100J -> Inductor_SMD:L_Wuerth_HCI-5040
Other:
- note added: "744766001"
Changed lines of the file:
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@@
+		)
+	)
+	(text "744766001"
+		(exclude_from_sim no)
+		(at 45.72 141.986 0)
+		(effects
+			(font
+				(size 1.27 1.27)
+			)
 		)
 	)
@@
 	)
 	(junction
-		(at 110.49 151.13)
-		(diameter 0)
-		(color 0 0 0 0)
-	)
-	(junction
 		(at 73.66 68.58)
 		(diameter 0)
@@
 	(wire
 		(pts
-			(xy 110.49 151.13) (xy 115.57 151.13)
+			(xy 106.68 151.13) (xy 115.57 151.13)
 		)
 		(stroke
@@
 		(pts
 			(xy 48.26 151.13) (xy 52.07 151.13)
-		)
-		(stroke
-			(width 0)
-			(type default)
-		)
-	)
-	(wire
-		(pts
-			(xy 106.68 151.13) (xy 110.49 151.13)
 		)
 		(stroke
@@
 			)
 		)
-		(property "Footprint" "Library_inductance_new:CWF1612A100J"
+		(property "Footprint" "Inductor_SMD:L_Wuerth_HCI-5040"
 			(at 45.72 151.13 0)
 			(effects
@@
 					(unit 1)
 				)
-			)
-		)
-	)
-	(symbol
-		(lib_id "Connector:TestPoint")
-		(at 110.49 151.13 0)
-		(unit 1)
-		(exclude_from_sim no)
-		(in_bom yes)
-		(on_board yes)
-		(dnp no)
-		(fields_autoplaced yes)
-		(property "Reference" "TP1"
-			(at 113.03 146.5579 0)
-			(effects
-				(font
-					(size 1.27 1.27)
-				)
-				(justify left)
-				(hide yes)
-			)
-		)
-		(property "Value" "TestPoint"
-			(at 113.03 149.0979 0)
-			(effects
-				(font
-					(size 1.27 1.27)
-				)
-				(justify left)
-				(hide yes)
-			)
-		)
-		(property "Footprint" "TestPoint:TestPoint_Pad_D1.5mm"
-			(at 115.57 151.13 0)
-			(effects
-				(font
-					(size 1.27 1.27)
-				)
-				(hide yes)
-			)
-		)
-		(property "Datasheet" "~"
-			(at 115.57 151.13 0)
-			(effects
-				(font
-					(size 1.27 1.27)
-				)
-				(hide yes)
-			)
-		)
-		(property "Description" "test point"
-			(at 110.49 151.13 0)
-			(effects
-				(font
-					(size 1.27 1.27)
-				)
-				(hide yes)
-			)
-		)
-		(pin "1"
-		)
-		(instances
-			(project "Enceinte"
-				(path "/7b437169-5795-4da0-84d7-3789a3b72d4c"
-					(reference "TP1")
-					(unit 1)
-				)
