File: Enceinte/TPA3110D2PWPR.kicad_sch (KiCad schematic)
At the start: 32 parts, among them IC1 TPA3110D2PWPR, J10 Conn_01x03, J11 Conn_01x03

Commit message: des changements sont à faire
Parts:
- C12, C19: footprint Capacitor_SMD:C_0603_1608Metric -> Capacitor_SMD:CP_Elec_6.3x7.7
Changed lines of the file:
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@@
 			)
 		)
-		(property "Footprint" "Capacitor_SMD:C_0603_1608Metric"
+		(property "Footprint" "Capacitor_SMD:CP_Elec_6.3x7.7"
 			(at 160.02 124.46 0)
 			(effects
@@
 			)
 		)
-		(property "Footprint" "Capacitor_SMD:C_0603_1608Metric"
+		(property "Footprint" "Capacitor_SMD:CP_Elec_6.3x7.7"
 			(at 121.92 43.18 0)
 			(effects

Commit message: doc latex
Parts:
- added TP3, TP4, TP5, TP6: TestPoint, TestPoint:TestPoint_Pad_D1.5mm, symbol Connector:TestPoint
- J10: renamed from J11; footprint Connector_PinSocket_2.54mm:PinSocket_1x03_P2.54mm_Vertical -> Connector_JST:JST_XH_B3B-XH-A_1x03_P2.50mm_Vertical
- J9: renamed from J10; footprint Connector_PinSocket_2.54mm:PinSocket_1x03_P2.54mm_Vertical -> Connector_JST:JST_XH_B3B-XH-A_1x03_P2.50mm_Vertical
- renumbered C8 to C10, C9 to C11, C10 to C12, C11 to C13, C12 to C14, C13 to C15, C14 to C16, C15 to C17, C16 to C18, C17 to C19, C18 to C20, C19 to C21, C20 to C22, C21 to C23, C22 to C24, C23 to C25, C24 to C26, C25 to C27, C5 to C7, C6 to C8, C7 to C9, L1 to L2, L2 to L3, L3 to L4, L4 to L5
Connections:
- net at C22.2, J9.1 (Pin_1), L2.2: now also TP3.1
- net at C23.2, J9.2 (Pin_2), L3.2: now also TP4.1
- net at C24.2, J10.1 (Pin_1), L4.2: now also TP5.1
- net at C25.2, J10.2 (Pin_2), L5.2: now also TP6.1

Commit message: nouvelles inductances
Parts:
- L2, L3, L4, L5: footprint Inductor_SMD:L_0603_1608Metric -> Library_inductance_new:SRN5040
Changed lines of the file:
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@@
 			)
 		)
-		(property "Footprint" "Inductor_SMD:L_0603_1608Metric"
+		(property "Footprint" "Library_inductance_new:SRN5040"
 			(at 162.56 73.66 0)
 			(effects
@@
 			)
 		)
-		(property "Footprint" "Inductor_SMD:L_0603_1608Metric"
+		(property "Footprint" "Library_inductance_new:SRN5040"
 			(at 162.56 88.9 0)
 			(effects
@@
 			)
 		)
-		(property "Footprint" "Inductor_SMD:L_0603_1608Metric"
+		(property "Footprint" "Library_inductance_new:SRN5040"
 			(at 162.56 114.3 0)
 			(effects
@@
 			)
 		)
-		(property "Footprint" "Inductor_SMD:L_0603_1608Metric"
+		(property "Footprint" "Library_inductance_new:SRN5040"
 			(at 162.56 99.06 0)
 			(effects

Commit message: indu Wurth
Parts:
- removed TP3, TP4, TP5, TP6: TestPoint, TestPoint:TestPoint_Pad_D1.5mm, symbol Connector:TestPoint
- L2, L3, L4, L5: footprint Library_inductance_new:SRN5040 -> Inductor_SMD:L_Wuerth_WE-PD-Typ-7345
Other:
- note added: "7447789115"
